File: ChillmonBoard.brd (EAGLE design)
At the start: 85 x 33.1 mm, 21 parts, among them J10 1X2-3.5MM, J11 1X2-3.5MM, J12 1X2-3.5MM, U1 MCP3008-I/SL, U2 ADR510ARTZ-REEL7

Commit message: Copied microBuilder Raspberry Pi shield, which I'd modified, to Chillmon.lbr
Parts:
- U$1: device microbuilder-ryan:RASBERRYPI_SHIELD -> Chillmon:RASBERRYPI_SHIELD
Changed lines of the file:
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@@
 <element name="J3" library="microbuilder" package="TERMBLOCK_1X3-3.5MM" value="" x="58.42" y="54.61"/>
 <element name="J4" library="microbuilder" package="TERMBLOCK_1X3-3.5MM" value="" x="46.99" y="54.61"/>
-<element name="U$1" library="microbuilder-ryan" package="RASBERRYPI_SHIELD" value="RASPBERRYPI_BB" x="21.59" y="-38.1" smashed="yes"/>
+<element name="U$1" library="Chillmon" package="RASBERRYPI_SHIELD" value="RASPBERRYPI_BB" x="21.59" y="-38.1" smashed="yes"/>
 <element name="J5" library="microbuilder" package="TERMBLOCK_1X3-3.5MM" value="" x="46.99" y="31.75" rot="R180"/>
 <element name="J6" library="microbuilder" package="TERMBLOCK_1X3-3.5MM" value="" x="58.42" y="31.75" rot="R180"/>

Commit message: Updated documentation for Rev1 vs. Rev2 Pi board changes. Added BOM.xls Made board a bit more pretty.
Parts:
- moved J10 1.27 mm to (8.89, 48.3)
- moved J11 0.63 mm to (8.89, 40.0)
Changed lines of the file:
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@@
 <text x="63.9064" y="59.7662" size="1.6764" layer="25" rot="R180">+</text>
 <text x="52.5272" y="59.7662" size="1.6764" layer="25" rot="R180">+</text>
-<text x="5.461" y="44.5262" size="1.6764" layer="25" rot="R180">+</text>
-<text x="5.4102" y="53.3654" size="1.6764" layer="25" rot="R180">+</text>
+<text x="5.461" y="43.8912" size="1.6764" layer="25" rot="R180">+</text>
+<text x="5.4102" y="52.0954" size="1.6764" layer="25" rot="R180">+</text>
 <text x="75.7428" y="26.6446" size="1.6764" layer="25">+</text>
 <text x="82.9818" y="43.5864" size="1.27" layer="25" rot="SR270">3.3V</text>
-<text x="34.29" y="48.26" size="1.778" layer="25">Chillmon v0.1</text>
-<text x="34.29" y="45.72" size="1.016" layer="25">(C) 2013 Ryan Pierce</text>
-<text x="34.29" y="44.45" size="1.016" layer="25">Licensed under CERN OHL v.1.1</text>
+<text x="31.75" y="48.26" size="1.778" layer="25">Chillmon v0.1</text>
+<text x="31.75" y="45.72" size="1.016" layer="25">(C) 2013 Ryan Pierce</text>
+<text x="31.75" y="44.45" size="1.016" layer="25">Licensed under CERN OHL v.1.1</text>
 <text x="24.13" y="35.56" size="1.27" layer="25">OneWire</text>
 <text x="13.97" y="38.1" size="1.27" layer="25" rot="R90">Outputs</text>
@@
 </element>
 <element name="R1" library="adafruit" package="R0805" value="4.7k" x="30.48" y="40.64"/>
-<element name="J10" library="adafruit" package="1X2-3.5MM" value="1X2-3.5MM" x="8.89" y="49.53" smashed="yes" rot="R90">
-<attribute name="NAME" x="4.2964" y="48.4152" size="0.8128" layer="25" rot="R270"/>
-</element>
-<element name="J11" library="adafruit" package="1X2-3.5MM" value="1X2-3.5MM" x="8.89" y="40.64" smashed="yes" rot="R90">
-<attribute name="NAME" x="4.2456" y="39.322" size="0.8128" layer="25" rot="R270"/>
+<element name="J10" library="adafruit" package="1X2-3.5MM" value="1X2-3.5MM" x="8.89" y="48.26" smashed="yes" rot="R90">
+<attribute name="NAME" x="4.2964" y="47.1452" size="0.8128" layer="25" rot="R270"/>
+</element>
+<element name="J11" library="adafruit" package="1X2-3.5MM" value="1X2-3.5MM" x="8.89" y="40.005" smashed="yes" rot="R90">
+<attribute name="NAME" x="4.2456" y="38.687" size="0.8128" layer="25" rot="R270"/>
 </element>
 <element name="J12" library="adafruit" package="1X2-3.5MM" value="1X2-3.5MM" x="8.89" y="31.75" smashed="yes" rot="R90">
 <attribute name="NAME" x="4.2964" y="30.5336" size="0.8128" layer="25" rot="R270"/>
 </element>
-<element name="R2" library="adafruit" package="R0805" value="10k" x="16.51" y="48.26"/>
-<element name="R3" library="adafruit" package="R0805" value="10k" x="21.59" y="48.26"/>
+<element name="R2" library="adafruit" package="R0805" value="10k" x="16.51" y="48.26" smashed="yes">
+<attribute name="NAME" x="16.0274" y="49.3014" size="1.27" layer="25"/>
+<attribute name="VALUE" x="15.748" y="45.974" size="1.27" layer="27"/>
+</element>
+<element name="R3" library="adafruit" package="R0805" value="10k" x="21.59" y="48.26" smashed="yes">
+<attribute name="NAME" x="20.828" y="49.276" size="1.27" layer="25"/>
+<attribute name="VALUE" x="20.701" y="45.9486" size="1.27" layer="27"/>
+</element>
 <element name="R4" library="adafruit" package="R0805" value="10k" x="26.67" y="46.99" smashed="yes" rot="R270">
-<attribute name="NAME" x="24.3586" y="48.2854" size="1.27" layer="25" rot="R270"/>
+<attribute name="NAME" x="24.3586" y="48.6156" size="1.27" layer="25" rot="R270"/>
 <attribute name="VALUE" x="27.8384" y="48.2092" size="1.27" layer="27" rot="R270"/>
 </element>
@@
 <attribute name="SUPPLIER" value="Analog Devices" x="80.01" y="46.99" size="1.778" layer="27" rot="R180" display="off"/>
 <attribute name="OC_FARNELL" value="-" x="80.01" y="46.99" size="1.778" layer="27" rot="R180" display="off"/>
-<attribute name="NAME" x="79.5528" y="45.5422" size="2.0828" layer="25" ratio="10" rot="SR270"/>
+<attribute name="NAME" x="79.1972" y="45.085" size="2.0828" layer="25" ratio="10" rot="SR270"/>
 <attribute name="VALUE" x="83.4644" y="51.435" size="2.0828" layer="48" ratio="10" rot="SR180"/>
 </element>
@@
 <contactref element="R2" pad="1"/>
 <contactref element="U$1" pad="11"/>
-<wire x1="19.05" y1="55.118" x2="15.262" y2="51.33" width="0.4064" layer="16"/>
-<wire x1="15.262" y1="51.33" x2="8.89" y2="51.33" width="0.4064" layer="16"/>
+<wire x1="19.05" y1="55.118" x2="15.262" y2="50.06" width="0.4064" layer="16"/>
+<wire x1="15.262" y1="50.06" x2="8.89" y2="50.06" width="0.4064" layer="16"/>
 <wire x1="15.51" y1="48.26" x2="15.262" y2="48.508" width="0.4064" layer="1"/>
-<wire x1="15.262" y1="48.508" x2="15.262" y2="51.33" width="0.4064" layer="1"/>
-<via x="15.262" y="51.33" extent="1-16" drill="0.6" shape="square"/>
+<wire x1="15.262" y1="48.508" x2="15.262" y2="50.06" width="0.4064" layer="1"/>
+<via x="15.262" y="50.06" extent="1-16" drill="0.6" shape="square"/>
 </signal>
 <signal name="CHILL2">
@@
 <wire x1="21.59" y1="55.118" x2="20.59" y2="54.118" width="0.4064" layer="1"/>
 <wire x1="20.59" y1="54.118" x2="20.59" y2="48.26" width="0.4064" layer="1"/>
-<wire x1="8.89" y1="42.44" x2="17.504" y2="42.4688" width="0.4064" layer="1"/>
-<wire x1="17.504" y1="42.4688" x2="20.5994" y2="45.72" width="0.4064" layer="16"/>
+<wire x1="8.89" y1="41.805" x2="16.6404" y2="41.7576" width="0.4064" layer="1"/>
+<wire x1="16.6404" y1="41.7576" x2="20.5994" y2="45.72" width="0.4064" layer="16"/>
 <wire x1="20.5994" y1="45.72" x2="20.59" y2="45.7294" width="0.4064" layer="1"/>
 <wire x1="20.59" y1="45.7294" x2="20.59" y2="48.26" width="0.4064" layer="1"/>
-<via x="17.504" y="42.4688" extent="1-16" drill="0.6" shape="square"/>
+<via x="16.6404" y="41.7576" extent="1-16" drill="0.6" shape="square"/>
 <via x="20.5994" y="45.72" extent="1-16" drill="0.6" shape="square"/>
 </signal>

Commit message: Changed routing of power to R1
Routing:
- net +3V3: track 243.1 -> 243.6 mm
Changed lines of the file:
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@@
 <layer number="47" name="Measures" color="7" fill="1" visible="yes" active="yes"/>
 <layer number="48" name="Document" color="7" fill="1" visible="no" active="yes"/>
-<layer number="49" name="Reference" color="7" fill="1" visible="yes" active="yes"/>
+<layer number="49" name="Reference" color="7" fill="1" visible="no" active="yes"/>
 <layer number="50" name="dxf" color="7" fill="1" visible="no" active="no"/>
 <layer number="51" name="tDocu" color="7" fill="1" visible="yes" active="yes"/>
@@
 <wire x1="24.39" y1="31.75" x2="24.384" y2="31.744" width="0.4064" layer="1"/>
 <wire x1="24.384" y1="31.744" x2="24.384" y2="29.0322" width="0.4064" layer="1"/>
-<wire x1="24.39" y1="31.75" x2="24.4" y2="36.82" width="0.4064" layer="1"/>
-<wire x1="24.4" y1="36.82" x2="29.48" y2="40.64" width="0.4064" layer="1"/>
 <wire x1="6.3246" y1="35.8394" x2="17.272" y2="35.8648" width="0.4064" layer="1"/>
-<wire x1="17.272" y1="35.8648" x2="24.13" y2="29.21" width="0.4064" layer="1"/>
+<wire x1="17.272" y1="35.8648" x2="20.89829375" y2="32.345953125" width="0.4064" layer="1"/>
 <contactref element="R5" pad="1"/>
+<wire x1="20.89829375" y1="32.345953125" x2="24.13" y2="29.21" width="0.4064" layer="1"/>
 <wire x1="73.93" y1="46.99" x2="73.9648" y2="48.6156" width="0.4064" layer="1"/>
 <wire x1="73.9648" y1="48.6156" x2="75.5556" y2="48.6156" width="0.4064" layer="1"/>
 <wire x1="75.5556" y1="48.6156" x2="76.47" y2="49.53" width="0.4064" layer="1"/>
 <wire x1="76.47" y1="49.53" x2="87.63" y2="49.53" width="0.4064" layer="1"/>
+<wire x1="29.48" y1="40.64" x2="20.89829375" y2="32.345953125" width="0.4064" layer="1"/>
 <wire x1="24.13" y1="29.21" x2="24.384" y2="29.0322" width="0" layer="19" extent="1-1"/>
 <wire x1="6.35" y1="35.9156" x2="6.3246" y2="35.8394" width="0" layer="19" extent="1-1"/>
